File: PCB/Flipklok/Flipklok.kicad_pcb (KiCad board)
At the start: 2 copper layers, 67 parts, among them J1 Power, J10 FW-btn, J11 RW-btn, J12 Programheader, J2 SW, J3 28BYJ-48, J4 Backlight, J5 DCF77, J6 LDR, J8 Indicator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

Commit message: Started optimizing routing and layout
Parts:
- removed R11: 1k, Resistor_SMD:R_0805_2012Metric_Pad1.20x1.40mm_HandSolder
- added H1: MountingHole_Pad, MountingHole:MountingHole_3.2mm_M3_DIN965_Pad_TopBottom, F.Cu at (121.7, 90.6)
- added H2: MountingHole_Pad, MountingHole:MountingHole_3.2mm_M3_DIN965_Pad_TopBottom, F.Cu at (66.5, 26.7)
- added H3: MountingHole_Pad, MountingHole:MountingHole_3.2mm_M3_DIN965_Pad_TopBottom, F.Cu at (114.7, 26.6)
- added H4: MountingHole_Pad, MountingHole:MountingHole_3.2mm_M3_DIN965_Pad_TopBottom, F.Cu at (66.7, 78.6)
- SW1: moved to F.Cu
- moved R17 216.3 mm to (71.7, 37.0), turned to -90 degrees
- moved R2 211.0 mm to (79.2, 42.7), turned to 0 degrees
- moved U2 210.2 mm to (74.6, 39.7), turned to 90 degrees
- moved R3 208.9 mm to (83.1, 42.7), turned to 0 degrees
- moved R1 208.7 mm to (81.9, 39.6), turned to -90 degrees
- moved D1 200.8 mm to (76.5, 34.7), turned to 90 degrees
- moved L1 177.8 mm to (81.4, 34.1), turned to 0 degrees
- moved C1 169.6 mm to (74.4, 34.9), turned to 90 degrees
- moved C3 167.3 mm to (77.7, 39.6), turned to 90 degrees
- moved C4 166.8 mm to (79.8, 39.6), turned to -90 degrees
- moved C2 160.3 mm to (84.0, 39.6), turned to -90 degrees
- moved R12 114.5 mm to (118.5, 63.2), turned to 90 degrees
- moved SW1 110.5 mm to (116.5, 62.4), turned to -90 degrees
- moved C10 108.7 mm to (116.5, 60.6), turned to 90 degrees
- moved R14 88.2 mm to (67.5, 86.2), turned to 0 degrees
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Connections:
- net IgnitionFB renamed IgnitionFB-A
- net Net-(D1-K) renamed /SW
- net Net-(U2-BST) renamed /BST
- net Net-(U2-FB) renamed /FB
- D3 pad 1: unconnected-(D3-IO1-Pad1) -> +5V
- D3 pad 4: +5V -> unconnected-(D3-IO3-Pad4)
- D6 pad 4: LDR -> Indicator
- D6 pad 5: Net-(J8-Pin_1) -> LDR-A
- D7 pad 4: RST/SBWTDIO -> TEST/SBWTCK
- D7 pad 5: TEST/SBWTCK -> RST/SBWTDIO
- D9 pad 3: +3.3V -> /DCF-A
- J3 pad 1: +5V -> Net-(J3-Pin_1)
- J3 pad 5: Net-(J3-Pin_5) -> +5V
- J5 pad 3: +3.3V -> /DCF-A
- J6 pad 1: LDR -> LDR-A
- J8 pad 1: Net-(J8-Pin_1) -> Indicator
- JP3 pad 1: +3.3V -> /DCF-A
- JP6 pad 2: BatteryFB -> BatteryFB-A
- R10 pad 2: LDR -> LDR-A
- R14 pad 1: +3.3V -> /DCF-A
- R4 pad 2: BatteryFB -> BatteryFB-A
- R5 pad 1: BatteryFB -> BatteryFB-A
- U1 pad 10: STEP-3 -> STEP-1
- U1 pad 12: Indicator -> STEP-3
- U1 pad 13: 5V-EN -> STEP-2
- U1 pad 15: DCF77 -> Indicator
- U1 pad 2: EN-pullup -> BatteryFB-A
- U1 pad 3: BatteryFB -> 5V-EN
- U1 pad 5: RW-btn -> EN-pullup
- U1 pad 6: FW-btn -> LDR-A
- U1 pad 7: LDR -> DCF77
- U1 pad 8: STEP-1 -> RW-btn
- U1 pad 9: STEP-2 -> FW-btn
- U5 pad 13: Net-(J3-Pin_5) -> Net-(J3-Pin_4)
- U5 pad 14: Net-(J3-Pin_4) -> Net-(J3-Pin_3)
- U5 pad 15: Net-(J3-Pin_3) -> Net-(J3-Pin_2)
- U5 pad 16: Net-(J3-Pin_2) -> Net-(J3-Pin_1)
Routing:
- net Net-(J11-Pin_1): track 0.00 -> 56.7 mm, vias 0 -> 2
- net Net-(J10-Pin_1): track 0.00 -> 56.5 mm, vias 0 -> 4
- net +3.3V: track 0.00 -> 53.3 mm, vias 0 -> 1
- net GND: track 0.00 -> 48.4 mm, vias 0 -> 100
- net IgnitionFB-A: track 0.00 -> 44.6 mm
- net Indicator: track 0.00 -> 40.0 mm, vias 0 -> 3
- net EN-pullup: track 0.00 -> 34.0 mm, vias 0 -> 2
- net 5V-EN: track 0.00 -> 33.7 mm, vias 0 -> 2
- net +12V: track 0.00 -> 33.2 mm
- net LDR-A: track 0.00 -> 32.8 mm, vias 0 -> 1
- net RST/SBWTDIO: track 0.00 -> 29.4 mm, vias 0 -> 3
- net TXD: track 0.00 -> 25.4 mm
- net +5V: track 0.00 -> 24.4 mm
- net BatteryFB-A: track 0.00 -> 23.6 mm, vias 0 -> 2
- net DCF77: track 0.00 -> 22.6 mm
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- added copper zone on B.Cu, net +12SW
- added copper zone on B.Cu, net +12V
- added copper zone on B.Cu, net +3.3V
- added copper zone on B.Cu, net +5V
- added copper zone on B.Cu, net /SW
- added copper zone on F.Cu, net GND
Other:
- board outline added: 70 x 72 mm
- rule pad_to_mask_clearance: 0 -> 0.038

Commit message: Finished lay-out and exported gerbers
Parts:
- J11: value RW-btn -> EX-btn
- JP6: moved to F.Cu
- moved R15 38.7 mm to (94.4, 88.0)
- moved J3 38.7 mm to (100.7, 60.5)
- moved C16 38.7 mm to (89.5, 85.4)
- moved D3 38.7 mm to (99.6, 76.1)
- moved J4 38.7 mm to (100.7, 81.7)
- moved JP5 38.7 mm to (82.7, 79.8)
- moved R13 38.7 mm to (94.4, 85.5)
- moved JP4 38.7 mm to (82.7, 77.3)
- moved U5 38.7 mm to (85.9, 64.6)
- moved D8 35.9 mm to (89.7, 68.3), turned to 90 degrees
- moved D7 34.5 mm to (95.1, 50.0), turned to 180 degrees
- moved J12 29.4 mm to (100.7, 38.6)
- moved R12 29.4 mm to (96.2, 44.0)
- moved Reset 29.4 mm to (94.2, 43.2)
- moved C10 29.0 mm to (94.2, 42.0)
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- renumbered SW1 to Reset
Connections:
- D7 pad 4: TEST/SBWTCK -> RST/SBWTDIO
- D7 pad 5: RST/SBWTDIO -> TEST/SBWTCK
- U1 pad 10: STEP-1 -> EX-btn
- U1 pad 2: BatteryFB-A -> 5V-EN
- U1 pad 3: 5V-EN -> BatteryFB-A
- U1 pad 8: RW-btn -> STEP-1
- U4 pad 8: RW-btn -> EX-btn
Routing:
- net +5V: track 24.4 -> 80.0 mm, vias 0 -> 1
- net +3.3V: track 53.3 -> 104.8 mm
- net BatteryFB-A: track 23.6 -> 66.1 mm, vias 2 -> 5
- net STEP-1: track 0.00 -> 23.5 mm
- net FW-btn: track 2.61 -> 23.7 mm
- net Backlight: track 0.00 -> 19.8 mm, vias 0 -> 1
- net STEP-4: track 0.00 -> 16.6 mm
- net RST/SBWTDIO: track 29.4 -> 45.3 mm, vias 3 -> 4
- net EX-btn: track 0.00 -> 14.3 mm
- net TEST/SBWTCK: track 19.9 -> 33.9 mm, vias 2 -> 0
- net 5V-EN: track 33.7 -> 21.2 mm
- net LDR-A: track 32.8 -> 20.9 mm
- net STEP-3: track 0.00 -> 11.1 mm
- net STEP-2: track 0.00 -> 11.1 mm
- net EN-pullup: track 34.0 -> 24.9 mm, vias 2 -> 3
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Other:
- board size 70 x 72 mm -> 48 x 72 mm
- board text added: "${ProjectName}"
- board text added: "12V+"
- board text added: "DCF77"
- board text added: "Designed by H.Buter"
- board text added: "EX-BTN"
- board text added: "FW-BTN"
- board text added: "LDR"
- board text added: "Light"
- board text added: "Power"
- board text added: "REV: ${REVISION}"
- board text added: "SBW"
- board text added: "Status"
- board text added: "Stepper"
- board text added: "Switched"
