File: PCB/Flipklok/Flipklok.kicad_sch (KiCad schematic)
At the start: 58 parts, among them J1 Power, J10 FW-btn, J11 RW-btn, J12 Programheader, J2 SW, J3 28BYJ-48 - 5V stepper, J4 Backlight, J5 DCF77, J6 LDR, J8 Indicator, SW1 Reset, U1 MSP430G2553IN20, U3 AP2205, U4 74HC00, U5 ULQ2003A, Y1 Crystal_Small

Commit message: Finished REV1.0 of schematic, started working on PCB
Parts:
- removed J5: DCF77, symbol Connector_Generic:Conn_01x03
- removed JP1: EN-RXD, symbol Jumper:SolderJumper_2_Open
- removed JP2: EN-TXD, symbol Jumper:SolderJumper_2_Open
- added C15, C16: 0.1uF, Capacitor_SMD:C_0805_2012Metric_Pad1.18x1.45mm_HandSolder, symbol Device:C
- added D9: ESDA5V3SC5, Package_TO_SOT_SMD:SOT-23-5, symbol Power_Protection:ESDA5V3SC5
- added J5: DCF77, Connector_JST:JST_XH_B4B-XH-A_1x04_P2.50mm_Vertical, symbol Connector_Generic:Conn_01x04
- added JP3: Bypass-LDF, Jumper:SolderJumper-2_P1.3mm_Open_Pad1.0x1.5mm, symbol Jumper:SolderJumper_2_Open
- added JP4, JP5: Bridged, Jumper:SolderJumper-2_P1.3mm_Bridged_Pad1.0x1.5mm, symbol Jumper:SolderJumper_2_Bridged
- added JP6: EN-RXD, Jumper:SolderJumper-2_P1.3mm_Open_Pad1.0x1.5mm, symbol Jumper:SolderJumper_2_Open
- added JP7: EN-TXD, Jumper:SolderJumper-2_P1.3mm_Open_Pad1.0x1.5mm, symbol Jumper:SolderJumper_2_Open
- added R15: R, Resistor_SMD:R_0805_2012Metric_Pad1.20x1.40mm_HandSolder, symbol Device:R
- added R16: 10k, Resistor_SMD:R_0805_2012Metric_Pad1.20x1.40mm_HandSolder, symbol Device:R
- added R17: 100k, Resistor_SMD:R_0805_2012Metric_Pad1.20x1.40mm_HandSolder, symbol Device:R
- C1, C10, C11, C14, C2, C3, C4, C5, C6, C7, C8, C9: footprint (none) -> Capacitor_SMD:C_0805_2012Metric_Pad1.18x1.45mm_HandSolder
- C12, C13: value C_Small -> C_x; footprint (none) -> Capacitor_SMD:C_0805_2012Metric_Pad1.18x1.45mm_HandSolder; now not fitted
- D1: footprint (none) -> Diode_SMD:D_SOD-123F
- D2: footprint (none) -> Package_TO_SOT_SMD:TSOT-23
- D4, D5: footprint (none) -> Diode_SMD:D_SMB_Handsoldering
- F2, F3: footprint (none) -> Fuse:Fuse_0603_1608Metric_Pad1.05x0.95mm_HandSolder
- J1, J10, J11, J2, J4, J6, J8: footprint (none) -> Connector_JST:JST_XH_B2B-XH-A_1x02_P2.50mm_Vertical
- J12: footprint (none) -> Connector_JST:JST_XH_B7B-XH-A_1x07_P2.50mm_Vertical
- J3: value 28BYJ-48 - 5V stepper -> 28BYJ-48; footprint (none) -> Connector_JST:JST_XH_B5B-XH-A_1x05_P2.50mm_Vertical
- L1: footprint (none) -> Inductor_SMD:L_Bourns_SRN6045TA
- R1, R10, R11, R12, R13, R14, R2, R3, R4, R5, R6, R7, R8, R9: footprint (none) -> Resistor_SMD:R_0805_2012Metric_Pad1.20x1.40mm_HandSolder
- SW1: footprint (none) -> Button_Switch_SMD:SW_Tactile_SPST_NO_Straight_CK_PTS636Sx25SMTRLFS
- U4: footprint (none) -> Package_SO:SOIC-14_3.9x8.7mm_P1.27mm
- U5: footprint (none) -> Package_DIP:DIP-16_W7.62mm_Socket_LongPads
- Y1: value Crystal_Small -> ECS-.327-6-13X; footprint (none) -> Crystal:Crystal_C26-LF_D2.1mm_L6.5mm_Horizontal
Connections:
- net +12SW: now also R17.1
- net +3.3V: now also C11.1, R14.1, U4.1, U4.10, U4.13, U4.14 (VCC), U4.4, C15.1, D9.1 (K), D9.3 (K), J5.1 (Pin_1), J5.3 (Pin_3), JP3.1 (A)
- net +5V: now also C16.1
- net 5V-EN: now also U1.13 (P2.5/TA1.2), R16.1, R17.2
- net Backlight: now also U1.14 (TDI/TCLK/UCB0SOMI/UCB0SCL/TA0.1/CA6/A6/P1.6)
- net BatteryFB: now also U1.3 (UCA0RXD/UCA0SOMI/TA0.0/CA1/A1/P1.1), JP6.2 (B)
- net EN-pullup: now also U1.2 (TA0CLK/ACLK/CA0/A0/P1.0); no longer U1.8 (P2.0/TA1.0)
- net FW-btn: now also U1.6 (TCK/SMCLK/UCB0STE/UCA0CLK/VREF+/VeREF+/CA4/A4/P1.4), U4.11; no longer D6.3 (K), J10.1 (Pin_1), R9.2, U1.10 (P2.2/TA1.1)
- net GND: now also C11.2, C14.2, U4.7 (GND), C15.2, C16.2, D9.2 (A), J5.2 (Pin_2), J5.4 (Pin_4), JP4.1 (A), JP5.1 (A), R16.2
- net IgnitionFB: now also U1.4 (UCA0TXD/UCA0SIMO/TA0.1/CA2/A2/P1.2), JP7.2 (B)
- net LDR: now also U1.7 (TMS/UCB0CLK/UCA0STE/TA0.0/CA5/A5/P1.5); no longer U1.11 (P2.3/TA1.0)
- net RW-btn: now also U1.5 (CAOUT/VREF-/VeREF-/CA3/A3/P1.3), U4.8; no longer D6.1 (K), J11.1 (Pin_1), R8.2, U1.9 (P2.1/TA1.1)
- net RXD: now also D7.1 (K), J12.4 (Pin_4), JP6.1 (A); no longer U1.3 (UCA0RXD/UCA0SOMI/TA0.0/CA1/A1/P1.1)
- net STEP-1: now also U1.8 (P2.0/TA1.0)
- net STEP-2: now also U1.9 (P2.1/TA1.1)
- net STEP-3: now also U1.10 (P2.2/TA1.1)
- net STEP-4: now also U1.11 (P2.3/TA1.0)
- net TXD: now also D7.3 (K), J12.5 (Pin_5), JP7.1 (A); no longer U1.4 (UCA0TXD/UCA0SIMO/TA0.1/CA2/A2/P1.2)
- net XIN: now also Y1.2; no longer Y1.1
- net XOUT: now also Y1.1; no longer Y1.2
- net DCF77: now reaches U1.15 (TDO/TDI/UCB0SIMO/UCB0SDA/CAOUT/CA7/A7/P1.7)
- net DCF77: now also U4.6
- net at J4.2 (Pin_2), R13.2: now also R15.2
- net at R14.2: now also C14.1, U4.2, JP3.2 (B)
- net at R13.1, U5.12 (O5): now also R15.1
- net at U5.6 (I6): now also JP4.2 (B)
- net at U5.7 (I7): now also JP5.2 (B)
- net at U4.5: now also U4.3
- net at U4.12: now also D6.3 (K), J10.1 (Pin_1), R9.2
- net at U4.9: now also D6.1 (K), J11.1 (Pin_1), R8.2
- no-connect marks 5 -> 7
Other:
- note added: "3.3V power"
- note added: "5.0V power"
- note added: "C_{L} = 0.5*C_{x} + C_{PCB} + C_{MCU} C_{PCB} = 2.5 pF PCB C_{L} must be 12.5 pF xtal datasheet C_{MCU} = 1, 6, 10, 12.5 pF based on BCSCTL3 register => C_{x} = (10-C_{MCU})*2 = 20 - 2 * C_{MCU} = 18, 8, 0 C_{x} = 0 when BCSCTL3(bits 3-2) = 10_{2} (10pF)"
- note added: "C_{o} =(L * ( I_{o} + ( I_{ripple} * 0.5)^{2})) / ((V_{ripple} + V_{o})^{2} - V_{o}^{2}) = (37u * ( 450m + ( 135m * 0.5)^{2})) / ((0.1 + 5)^{2} - 5^{2}) = 10uF"
- note added: "Crystal LF"
- note added: "DCF including filtering"
- note added: "Forward and rewind buttons, Light sensor and indicator light"
- note added: "I_{ripple} = 0.3 * I_{max} = 0.3 * 450m = 135mA L=(V_{o} * (V_{i}-V_{o}))/(V_{i}* I_{ripple} * f_{sw})=(5 *(12-5))(5 * 0.135 * 1.4M) = 37uH => L = 33uH"
- note added: "LDF f_c ="
- note added: "Logic power"
- note added: "Power input"
- note added: "Power status"
- note added: "Programming"
- note added: "Reset-BTN"
- note added: "Stepper and backlight driver"
- note added: "V_{o} = (R1/(R2+R3)+1)*0.81= (${/02bf3ab9-1c95-4b58-ba06-e652d38e350a/d6bb5f7a-a4dc-4308-b162-b9847f2d8f0e:value}/(${/02bf3ab9-1c95-4b58-ba06-e652d38e350a/5491f8df-bb1c-4095-bf22-26e5e74846ff:value}+${/02bf3ab9-1c95-4b58-ba06-e652d38e350a/69f8bb98-a694-47f6-9a6b-2e9b63e3355e:value}) + 1) * 0.81 = 5.0952V"
- company: (none) -> Hogeschool Windesheim
- title: (none) -> ${ProjectName}
- moved on the sheet: C1, C10, C11, C14, C2, C3, C4, C5, C6, D1, D2, D3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

Commit message: Started optimizing routing and layout
Parts:
- removed R11: 1k, Resistor_SMD:R_0805_2012Metric_Pad1.20x1.40mm_HandSolder, symbol Device:R
- added H1, H2, H3, H4: MountingHole_Pad, MountingHole:MountingHole_3.2mm_M3_DIN965_Pad_TopBottom, symbol Mechanical:MountingHole_Pad
Connections:
- net +3.3V: no longer D9.3 (K), J5.3 (Pin_3), JP3.1 (A), R14.1
- net +5V: now also D3.1 (IO1), J3.5 (Pin_5); no longer D3.4 (IO3), J3.1 (Pin_1)
- net 5V-EN: now also U1.3 (UCA0RXD/UCA0SOMI/TA0.0/CA1/A1/P1.1); no longer U1.13 (P2.5/TA1.2)
- net DCF77: now also U1.7 (TMS/UCB0CLK/UCA0STE/TA0.0/CA5/A5/P1.5); no longer U1.15 (TDO/TDI/UCB0SIMO/UCB0SDA/CAOUT/CA7/A7/P1.7)
- net EN-pullup: now also U1.5 (CAOUT/VREF-/VeREF-/CA3/A3/P1.3); no longer U1.2 (TA0CLK/ACLK/CA0/A0/P1.0)
- net FW-btn: now also U1.9 (P2.1/TA1.1); no longer U1.6 (TCK/SMCLK/UCB0STE/UCA0CLK/VREF+/VeREF+/CA4/A4/P1.4)
- net GND: now also H1.1, H2.1, H3.1, H4.1
- net Indicator: now also D6.4 (K), J8.1 (Pin_1), U1.15 (TDO/TDI/UCB0SIMO/UCB0SDA/CAOUT/CA7/A7/P1.7); no longer U1.12 (P2.4/TA1.2)
- net RST/SBWTDIO: now also D7.5 (K); no longer D7.4 (K)
- net RW-btn: now also U1.8 (P2.0/TA1.0); no longer U1.5 (CAOUT/VREF-/VeREF-/CA3/A3/P1.3)
- net STEP-1: now also U1.10 (P2.2/TA1.1); no longer U1.8 (P2.0/TA1.0)
- net STEP-2: now also U1.13 (P2.5/TA1.2); no longer U1.9 (P2.1/TA1.1)
- net STEP-3: now also U1.12 (P2.4/TA1.2); no longer U1.10 (P2.2/TA1.1)
- net TEST/SBWTCK: now also D7.4 (K); no longer D7.5 (K)
- net FB: now reaches C4.2, R1.2, R2.1, U2.3 (FB)
- net SW: now reaches C3.2, D1.1 (K), L1.1, U2.6 (SW)
- net LDR-A: now reaches D6.5 (K)
- net LDR-A: now also J6.1 (Pin_1), R10.2, U1.6 (TCK/SMCLK/UCB0STE/UCA0CLK/VREF+/VeREF+/CA4/A4/P1.4); no longer J8.1 (Pin_1)
- net at U5.16 (O1): now also J3.1 (Pin_1); no longer J3.2 (Pin_2)
- net at U5.15 (O2): now also J3.2 (Pin_2); no longer J3.3 (Pin_3)
- net at U5.14 (O3): now also J3.3 (Pin_3); no longer J3.4 (Pin_4)
- net at U5.13 (O4): now also J3.4 (Pin_4); no longer J3.5 (Pin_5)
- net BST: now reaches C3.1, U2.1 (BST)
- net BatteryFB renamed BatteryFB-A
- net BatteryFB-A: now also U1.2 (TA0CLK/ACLK/CA0/A0/P1.0); no longer U1.3 (UCA0RXD/UCA0SOMI/TA0.0/CA1/A1/P1.1)
- net IgnitionFB renamed IgnitionFB-A
- removed net LDR: D6.4 (K), J6.1 (Pin_1), R10.2, U1.7 (TMS/UCB0CLK/UCA0STE/TA0.0/CA5/A5/P1.5)
- new net DCF-A: D9.3 (K), J5.3 (Pin_3), JP3.1 (A), R14.1
Other:
- note removed: "Indcator LED Vf = 2.5V@1mA Ur = 3.3-2.5 = 0.8V R = UR/IL = 0.8/1m = 800 ohm => 1k"
- moved on the sheet: C2, C5, C6, D3, J3, J4, JP6, JP7, R13, R15, R16, U3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

Commit message: Finished lay-out and exported gerbers
Parts:
- J11: value RW-btn -> EX-btn
Connections:
- net 5V-EN: now also U1.2 (TA0CLK/ACLK/CA0/A0/P1.0); no longer U1.3 (UCA0RXD/UCA0SOMI/TA0.0/CA1/A1/P1.1)
- net BatteryFB-A: now also U1.3 (UCA0RXD/UCA0SOMI/TA0.0/CA1/A1/P1.1); no longer U1.2 (TA0CLK/ACLK/CA0/A0/P1.0)
- net RST/SBWTDIO: now also D7.4 (K); no longer D7.5 (K)
- net STEP-1: now also U1.8 (P2.0/TA1.0); no longer U1.10 (P2.2/TA1.1)
- net TEST/SBWTCK: now also D7.5 (K); no longer D7.4 (K)
- net RW-btn renamed EX-btn
- net EX-btn: now also U1.10 (P2.2/TA1.1); no longer U1.8 (P2.0/TA1.0)
