File: PCB/Flipklok/Flipklok.kicad_sch (KiCad schematic)
At the start: 70 parts, among them J1 Power, J10 FW-btn, J11 EX-btn, J12 Programheader, J2 SW, J3 28BYJ-48, J4 Backlight, J5 DCF77, J6 LDR, J8 Indicator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

Commit message: filled in "to be detriment values" and updated BOM
Parts:
- C12, C13, R15: now left out of the parts list
- C14: value C -> 100n
- R13: value R -> 470
- R14: value R -> 10k
- R4, R6: value R -> 75k
- R5, R7: value R -> 18k
Other:
- note added: "LPF f_c = 2 * pi * 10k * 100n = 159 Hz"
- note added: "U_max = 16V Uo = 18/(18+75)*16=3.1V"
- note removed: "LDF f_c ="
Changed lines of the file:
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@@
 	(rectangle
 		(start 12.7 77.47)
-		(end 54.61 113.03)
+		(end 67.31 113.03)
 		(stroke
 			(width 0)
@@
 	(text "Power status\n"
 		(exclude_from_sim no)
-		(at 54.61 78.74 0)
+		(at 67.31 78.74 0)
 		(effects
 			(font
@@
 		)
 	)
-	(text "LDF\nf_c = \n"
+	(text "LPF\nf_c = 2 * pi * 10k * 100n = 159 Hz\n"
 		(exclude_from_sim no)
-		(at 80.01 259.08 0)
+		(at 73.66 261.62 0)
 		(effects
 			(font
 				(size 1.27 1.27)
 			)
+			(justify left)
 		)
 	)
@@
 		)
 	)
+	(text "U_max = 16V\nUo = 18/(18+75)*16=3.1V"
+		(exclude_from_sim no)
+		(at 39.37 110.49 0)
+		(effects
+			(font
+				(size 1.27 1.27)
+			)
+			(justify left)
+		)
+	)
 	(text "V_{o} = (R1/(R2+R3)+1)*0.81=  (${/02bf3ab9-1c95-4b58-ba06-e652d38e350a/d6bb5f7a-a4dc-4308-b162-b9847f2d8f0e:value}/(${/02bf3ab9-1c95-4b58-ba06-e652d38e350a/5491f8df-bb1c-4095-bf22-26e5e74846ff:value}+${/02bf3ab9-1c95-4b58-ba06-e652d38e350a/69f8bb98-a694-47f6-9a6b-2e9b63e3355e:value}) + 1) * 0.81 = 5.0952V"
 		(exclude_from_sim no)
@@
 		(polyline
 			(pts
-				(xy 142.24 83.82) (xy 184.15 83.82) (xy 184.15 107.95) (xy 142.24 107.95)
+				(xy 13.97 13.97) (xy 62.23 13.97) (xy 62.23 71.12) (xy 13.97 71.12) (xy 13.97 15.24)
 			)
 			(stroke
@@
 		(polyline
 			(pts
-				(xy 402.59 16.51) (xy 339.09 16.51) (xy 339.09 71.12) (xy 402.59 71.12)
+				(xy 163.83 233.68) (xy 130.81 233.68) (xy 130.81 273.05) (xy 163.83 273.05)
 			)
 			(stroke
@@
 		(polyline
 			(pts
-				(xy 13.97 13.97) (xy 62.23 13.97) (xy 62.23 71.12) (xy 13.97 71.12) (xy 13.97 15.24)
+				(xy 196.85 13.97) (xy 237.49 13.97) (xy 237.49 38.1) (xy 196.85 38.1)
 			)
 			(stroke
@@
 		(polyline
 			(pts
-				(xy 163.83 233.68) (xy 130.81 233.68) (xy 130.81 273.05) (xy 163.83 273.05)
+				(xy 142.24 83.82) (xy 184.15 83.82) (xy 184.15 107.95) (xy 142.24 107.95)
 			)
 			(stroke
@@
 		(polyline
 			(pts
-				(xy 196.85 13.97) (xy 237.49 13.97) (xy 237.49 38.1) (xy 196.85 38.1)
+				(xy 402.59 16.51) (xy 339.09 16.51) (xy 339.09 71.12) (xy 402.59 71.12)
 			)
 			(stroke
@@
 			)
 		)
-		(property "Value" "R"
+		(property "Value" "18k"
 			(at 38.1 102.8699 0)
 			(effects
@@
 			)
 		)
-		(property "Value" "R"
+		(property "Value" "75k"
 			(at 38.1 92.7099 0)
 			(effects
@@
 			)
 		)
-		(property "Value" "R"
+		(property "Value" "10k"
 			(at 59.69 252.73 90)
 			(effects
@@
 			)
 		)
-		(property "Value" "C"
+		(property "Value" "100n"
 			(at 73.66 256.5399 0)
 			(effects
@@
 		(unit 1)
 		(exclude_from_sim no)
-		(in_bom yes)
+		(in_bom no)
 		(on_board yes)
 		(dnp yes)
@@
 		(unit 1)
 		(exclude_from_sim no)
-		(in_bom yes)
+		(in_bom no)
 		(on_board yes)
 		(dnp yes)
@@
 		(unit 1)
 		(exclude_from_sim no)
-		(in_bom yes)
+		(in_bom no)
 		(on_board yes)
 		(dnp yes)
@@
 			)
 		)
-		(property "Value" "R"
+		(property "Value" "18k"
 			(at 20.32 102.8699 0)
 			(effects
@@
 			)
 		)
-		(property "Value" "R"
-			(at 361.95 41.91 90)
+		(property "Value" "470"
+			(at 363.22 41.91 90)
 			(effects
 				(font
@@
 			)
 		)
-		(property "Value" "R"
+		(property "Value" "75k"
 			(at 20.32 92.7099 0)
 			(effects
